Commit message: removed dependency on uuv_sim

File: potrov2_description/urdf/sensors.xacro (robot description, xacro)
@@ -24,3 +24,13 @@
     <origin xyz="0 0 0" rpy="0 0 0"/>
   </xacro:default_pressure>
+  <!-- DVL  -->
+  <xacro:default_dvl_macro
+    namespace="${namespace}"
+    parent_link="${namespace}/base_link"
+    inertial_reference_frame="world">
+    <origin xyz="0 0 0" rpy="0 1.57079 0"/>
+  </xacro:default_dvl_macro>
+  <!-- RPT  -->
+   <!-- Mount a GPS. -->
+  <xacro:default_gps namespace="${namespace}" parent_link="${namespace}/base_link" />
 </robot>
